Commit message: Update:Cartographer

File: src/fishbot_description/urdf/fishbot_base.urdf (robot description, URDF)
Before this commit: robot fishbot, 6 links, 5 joints
Links:
- removed link laser_link
- added link laser; visual cylinder length=0.02 radius=0.02
Joints:
- joint laser_joint: child laser_link -> laser
